Commit message: fixed wheels under going issue

File: ros_ws/src/nexzino/urdf/nexzino.urdf.xacro (robot description, xacro)
@@ -55,5 +55,14 @@
   </link>
   <joint name="base_footprint_joint" type="fixed">
-    <origin xyz="0 0 0" rpy="0 0 0" />
+    <!-- base_footprint is supposed to sit at true ground level (REP-120) -
+         this was identity, coinciding exactly with base_link, but base_link
+         isn't at ground height: the wheel joints mount at z=-0.014999
+         relative to base_link (see leftwheel_joint/rightwheel_joint below),
+         and diff_drive.yaml's wheel_radius is 0.105, so true wheel-ground
+         contact is at base_link z = -0.014999 - 0.105 =~ -0.12. Offsetting
+         base_link up by 0.12 here puts base_footprint's z=0 back at actual
+         ground level, matching what RTAB-Map/move_base assume "ground"
+         means for a base_footprint-framed grid/costmap. -->
+    <origin xyz="0 0 0.12" rpy="0 0 0" />
     <parent link="base_footprint" />
     <child link="base_link" />

Commit message: merging urdf

File: ros_ws/src/nexzino/urdf/nexzino.urdf.xacro (robot description, xacro)
@@ -1,67 +1,23 @@
-<?xml version="1.0" encoding="utf-8"?>
-<!-- This URDF was automatically created by SolidWorks to URDF Exporter! Originally created by Stephen Brawner (brawner@gmail.com)
-     Commit Version: 1.6.0-1-g15f4949  Build Version: 1.6.7594.29634
-     For more information, please see http://wiki.ros.org/sw_urdf_exporter -->
-<robot
-  name="nexzino"
-  xmlns:xacro="http://ros.org/wiki/xacro">
+<?xml version="1.0"?>
+<robot xmlns:xacro="http://ros.org/wiki/xacro"
+  name="nexzino">
   <xacro:arg name="use_gazebo" default="false" />
   <xacro:arg name="publish_pointcloud" default="true" />
-  <xacro:arg name="use_nominal_extrinsics" default="true" />
+  <!-- Default flipped from true: the depth/color/optical frame chain now
+       comes from the live realsense2_camera driver's real calibrated
+       extrinsics (publish_tf:=true in realsense_bringup.launch) instead of
+       static guessed numbers. Still overridable to true for offline
+       display.launch/Gazebo use where no driver is running to publish
+       those frames dynamically. -->
+  <xacro:arg name="use_nominal_extrinsics" default="false" />
   <xacro:include filename="$(find realsense2_description)/urdf/_d435.urdf.xacro" />
   <xacro:include filename="$(find nexzino)/urdf/nexzino.gazebo.xacro" />
-  <link
-    name="base_footprint">
-  </link>
-  <link
-    name="base_link">
-    <inertial>
-      <origin
-        xyz="0.023363 4.2288E-05 0.048586"
-        rpy="0 0 0" />
-      <mass
-        value="2.6736" />
-      <inertia
-        ixx="0.083868"
-        ixy="-4.2036E-06"
-        ixz="0.0012949"
-        iyy="0.09527"
-        iyz="1.6066E-06"
-        izz="0.040948" />
-    </inertial>
-    <visual>
-      <origin
-        xyz="0 0 0"
-        rpy="0 0 0" />
-      <geometry>
-        <mesh
-          filename="package://nexzino/meshes/base_link.STL" />
-      </geometry>
-      <material
-        name="">
-        <color
-          rgba="0.5098 0.5098 0.5098 1" />
-      </material>
-    </visual>
-    <collision>
-      <origin
-        xyz="0 0 0"
-        rpy="0 0 0" />
-      <geometry>
-        <mesh
-          filename="package://nexzino/meshes/base_link.STL" />
-      </geometry>
-    </collision>
-  </link>
+  <link name="base_footprint"></link>
   <joint name="base_footprint_joint" type="fixed">
-    <!-- base_footprint is supposed to sit at true ground level (REP-120) -
-         this was identity, coinciding exactly with base_link, but base_link
-         isn't at ground height: the wheel joints mount at z=-0.014999
-         relative to base_link (see leftwheel_joint/rightwheel_joint below),
-         and diff_drive.yaml's wheel_radius is 0.105, so true wheel-ground
-         contact is at base_link z = -0.014999 - 0.105 =~ -0.12. Offsetting
-         base_link up by 0.12 here puts base_footprint's z=0 back at actual
-         ground level, matching what RTAB-Map/move_base assume "ground"
-         means for a base_footprint-framed grid/costmap. -->
+    <!-- base_footprint sits at true ground level (REP-120): wheel joints
+         mount at z=-0.014999 relative to base_link, and diff_drive.yaml's
+         wheel_radius is 0.105, so true wheel-ground contact is at base_link
+         z = -0.014999 - 0.105 =~ -0.12. Offsetting base_link up by 0.12
+         here puts base_footprint's z=0 back at actual ground level. -->
     <origin xyz="0 0 0.12" rpy="0 0 0" />
     <parent link="base_footprint" />
@@ -69,18 +25,58 @@
   </joint>
   <link
+    name="base_link">
+    <inertial>
+      <origin
+        xyz="0.0233629429238116 4.22881594878133E-05 0.0485862192692521"
+        rpy="0 0 0" />
+      <mass
+        value="2.67357451448379" />
+      <inertia
+        ixx="0.0838676214813811"
+        ixy="-4.20361720258225E-06"
+        ixz="0.00129491227389105"
+        iyy="0.0952701211607136"
+        iyz="1.6066275313901E-06"
+        izz="0.0409475340600111" />
+    </inertial>
+    <visual>
+      <origin
+        xyz="0 0 0"
+        rpy="0 0 0" />
+      <geometry>
+        <mesh
+          filename="package://nexzino/meshes/base_link.STL" />
+      </geometry>
+      <material
+        name="">
+        <color
+          rgba="0.509803921568627 0.509803921568627 0.509803921568627 1" />
+      </material>
+    </visual>
+    <collision>
+      <origin
+        xyz="0 0 0"
+        rpy="0 0 0" />
+      <geometry>
+        <mesh
+          filename="package://nexzino/meshes/base_link.STL" />
+      </geometry>
+    </collision>
+  </link>
+  <link
     name="leftwheel_link">
     <inertial>
       <origin
-        xyz="-1.7408E-10 1.7408E-10 0.00038157"
-        rpy="0 0 0" />
-      <mass
-        value="1.4492" />
-      <inertia
-        ixx="0.0034708"
-        ixy="-5.8845E-16"
-        ixz="-1.2916E-09"
-        iyy="0.0034708"
-        iyz="1.2916E-09"
-        izz="0.0063018" />
+        xyz="-1.74075753811564E-10 1.74083775172917E-10 0.000381565663131411"
+        rpy="0 0 0" />
+      <mass
+        value="1.44920481477612" />
+      <inertia
+        ixx="0.00347079630181746"
+        ixy="-5.8844939595754E-16"
+        ixz="-1.29155431134988E-09"
+        iyy="0.00347079630181747"
+        iyz="1.29155395907396E-09"
+        izz="0.00630183667634335" />
     </inertial>
     <visual>
@@ -95,13 +91,14 @@
         name="">
         <color
-          rgba="0.21569 0.21569 0.21569 1" />
-      </material>
-    </visual>
-    <collision>
-      <origin
-        xyz="0 0 0"
-        rpy="0 0 0" />
-      <geometry>
-        <cylinder radius="0.105" length="0.05" />
+          rgba="0.215686274509804 0.215686274509804 0.215686274509804 1" />
+      </material>
+    </visual>
+    <collision>
+      <origin
+        xyz="0 0 0"
+        rpy="0 0 0" />
+      <geometry>
+        <mesh
+          filename="package://nexzino/meshes/leftwheel_link.STL" />
       </geometry>
     </collision>
@@ -111,6 +108,6 @@
     type="continuous">
     <origin
-      xyz="0.054039 0.16978 -0.014999"
-      rpy="1.5708 0 0" />
+      xyz="0.0540389524650898 0.169779999524495 -0.0149989847207889"
+      rpy="1.5707963267949 0 0" />
     <parent
       link="base_link" />
@@ -118,408 +115,376 @@
       link="leftwheel_link" />
     <axis
+      xyz="0 0 0.999999999999792" />
+  </joint>
+  <link
+    name="rightwheel_link">
+    <inertial>
+      <origin
+        xyz="1.74075198700052E-10 -1.74083469861586E-10 -0.000381565663131717"
+        rpy="0 0 0" />
+      <mass
+        value="1.44920481477613" />
+      <inertia
+        ixx="0.00347079630181749"
+        ixy="-5.88843528628314E-16"
+        ixz="-1.29155425553129E-09"
+        iyy="0.00347079630181749"
+        iyz="1.2915540535382E-09"
+        izz="0.00630183667634338" />
+    </inertial>
+    <visual>
+      <origin
+        xyz="0 0 0"
+        rpy="0 0 0" />
+      <geometry>
+        <mesh
+          filename="package://nexzino/meshes/rightwheel_link.STL" />
+      </geometry>
+      <material
+        name="">
+        <color
+          rgba="0.215686274509804 0.215686274509804 0.215686274509804 1" />
+      </material>
+    </visual>
+    <collision>
+      <origin
+        xyz="0 0 0"
+        rpy="0 0 0" />
+      <geometry>
+        <mesh
+          filename="package://nexzino/meshes/rightwheel_link.STL" />
+      </geometry>
+    </collision>
+  </link>
+  <joint
+    name="rightwheel_joint"
+    type="continuous">
+    <origin
+      xyz="0.0540387975537798 -0.169780000237316 -0.0149988298094792"
+      rpy="1.5707963267949 0 0" />
+    <parent
+      link="base_link" />
+    <child
+      link="rightwheel_link" />
+    <axis
+      xyz="0 0 0.999999999999792" />
+  </joint>
+  <link
+    name="casterwheelmount_link">
+    <inertial>
+      <origin
+        xyz="0.00187352191273216 0.0129405492524937 -0.0103000078506701"
+        rpy="0 0 0" />
+      <mass
+        value="0.0102706017023182" />
+      <inertia
+        ixx="3.93968493623888E-06"
+        ixy="-2.8232800941337E-07"
+        ixz="5.63131676132563E-08"
+        iyy="3.432191688351E-06"
+        iyz="1.42222659679423E-06"
+        izz="3.85767367428349E-06" />
+    </inertial>
+    <visual>
+      <origin
+        xyz="0 0 0"
+        rpy="0 0 0" />
+      <geometry>
+        <mesh
+          filename="package://nexzino/meshes/casterwheelmount_link.STL" />
+      </geometry>
+      <material
+        name="">
+        <color
+          rgba="0.509803921568627 0.509803921568627 0.509803921568627 1" />
+      </material>
+    </visual>
+    <collision>
+      <origin
+        xyz="0 0 0"
+        rpy="0 0 0" />
+      <geometry>
+        <mesh
+          filename="package://nexzino/meshes/casterwheelmount_link.STL" />
+      </geometry>
+    </collision>
+  </link>
+  <joint
+    name="casterwheelmount_joint"
+    type="continuous">
+    <origin
+      xyz="0.139639576281008 0.0791060227155972 -0.051842999999996"
+      rpy="-1.5707963267949 0 -1.5707963267949" />
+    <parent
+      link="base_link" />
+    <child
+      link="casterwheelmount_link" />
+    <axis
+      xyz="0 -1 0" />
+  </joint>
+  <link
+    name="casterwheel_link">
+    <inertial>
+      <origin
+        xyz="1.33226762955019E-15 1.23512311489549E-15 -0.0112773964520611"
+        rpy="0 0 0" />
+      <mass
+        value="0.0399331188999233" />
+      <inertia
+        ixx="7.77541411629872E-06"
+        ixy="-1.01833774330127E-21"
+        ixz="-2.72426971660664E-19"
+        iyy="7.77541411629871E-06"
+        iyz="4.13954478132233E-19"
+        izz="1.27535117768465E-05" />
+    </inertial>
+    <visual>
+      <origin
+        xyz="0 0 0"
+        rpy="0 0 0" />
+      <geometry>
+        <mesh
+          filename="package://nexzino/meshes/casterwheel_link.STL" />
+      </geometry>
+      <material
+        name="">
+        <color
+          rgba="0.270588235294118 0.270588235294118 0.270588235294118 1" />
+      </material>
+    </visual>
+    <collision>
+      <origin
+        xyz="0 0 0"
+        rpy="0 0 0" />
+      <geometry>
+        <mesh
+          filename="package://nexzino/meshes/casterwheel_link.STL" />
+      </geometry>
+    </collision>
+  </link>
+  <joint
+    name="casterwheel_joint"
+    type="continuous">
+    <origin
+      xyz="0.0151109163570423 0.0349719999999999 -0.0235537261563978"
+      rpy="0 -1.41616610057807 3.14159265358979" />
+    <parent
+      link="casterwheelmount_link" />
+    <child
+      link="casterwheel_link" />
+    <axis
+      xyz="-3.74938274523284E-05 0 -0.999999999297106" />
+  </joint>
+  <link
+    name="casterwheelmount1_link">
+    <inertial>
+      <origin
+        xyz="-0.0101545114856474 0.00254678088783966 0.0129405492213775"
+        rpy="0 0 0" />
+      <mass
+        value="0.0102706060663648" />
+      <inertia
+        ixx="3.86541891392595E-06"
+        ixy="6.12075400190165E-08"
+        ixz="1.40058301400974E-06"
+        iyy="3.93194090481684E-06"
+        iyz="-3.75240720638479E-07"
+        izz="3.43219229056267E-06" />
+    </inertial>
+    <visual>
+      <origin
+        xyz="0 0 0"
+        rpy="0 0 0" />
+      <geometry>
+        <mesh
+          filename="package://nexzino/meshes/casterwheelmount1_link.STL" />
+      </geometry>
+      <material
+        name="">
+        <color
+          rgba="0.509803921568627 0.509803921568627 0.509803921568627 1" />
+      </material>
+    </visual>
+    <collision>
+      <origin
+        xyz="0 0 0"
+        rpy="0 0 0" />
+      <geometry>
+        <mesh
+          filename="package://nexzino/meshes/casterwheelmount1_link.STL" />
+      </geometry>
+    </collision>
+  </link>
+  <joint
+    name="casterwheelmount1_joint"
+    type="continuous">
+    <origin
+      xyz="0.139639576281007 -0.0808939772844029 -0.051842999999996"
+      rpy="-3.14159265358979 0 0" />
+    <parent
+      link="base_link" />
+    <child
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
Commit message: realsense orientation 1

File: ros_ws/src/nexzino/urdf/nexzino.urdf.xacro (robot description, xacro)
@@ -700,41 +700,26 @@
       xyz="0 0 0" />
   </joint>
-  <!-- camera_tilt_link re-establishes standard camera-body convention
-       (X=forward, Y=left, Z=up) on top of realsense_Link's own frame - this
-       exact rotation (1.5708, 3.1416, 3.1416) is the one already proven, by
-       explicit rotation-matrix calculation, to make a camera attached here
-       read out exactly forward-level (see conversation history / git log
-       for the derivation). It is NOT a guess.
-       camera_tilt_pitch below is the one remaining unknown: the physical
-       camera is mounted tilted down by some angle, confirmed by loading the
-       real CAD mesh (nexa package) - a plain screenshot comparison isn't
-       precise enough to read off the exact angle, so this defaults to 0
-       (matches the old, forward-level behavior) rather than guessing a
-       number. To find the real value: watch nav_console's live camera feed
-       (or RViz's point cloud) while adjusting this, positive tilts the
-       camera further DOWN (confirmed: positive pitch about Y in this frame
-       rotates +X toward -Z). Try increments like 0.2-0.5 (≈11-29°) and
-       rebuild until the floor fills the frame the way it does on the real
-       robot. -->
-  <xacro:property name="camera_tilt_pitch" value="0" />
-  <link name="camera_tilt_link" />
-  <joint name="camera_tilt_joint" type="fixed">
-    <origin xyz="0 0 0" rpy="1.5708 3.1416 3.1416" />
-    <parent link="realsense_Link" />
-    <child link="camera_tilt_link" />
-  </joint>
-  <!-- Depth/color/optical frame orientations come from the live camera
-       driver's own calibrated extrinsics (see realsense_bringup.launch's
-       publish_tf:=true / use_nominal_extrinsics:=false), not from static
-       numbers here - use_nominal_extrinsics is kept as a fallback for
-       offline display/Gazebo use where no live driver is publishing those
-       frames. -->
+  <!-- Camera sensor frames attached directly at realsense_Link's own pose -
+       zero extra rotation, zero extra offset. realsense_Link's mesh (a
+       combined mount-arm + camera unit, confirmed visually against the
+       real robot) IS the ground truth for where/how the camera sits; no
+       hand-derived compensating rotation on top of it. (An earlier attempt
+       to derive that compensating rotation mathematically produced a
+       provably wrong result - the mesh mixes mount-arm and camera geometry,
+       so its own axes can't be read off computationally either. This is
+       the deliberate alternative: trust the CAD pose completely instead of
+       guessing a correction for it.)
+       Depth/color/optical frame orientations still come from the live
+       camera driver's own calibrated extrinsics (realsense_bringup.launch's
+       publish_tf:=true / use_nominal_extrinsics:=false), not static numbers
+       here - use_nominal_extrinsics is kept as a fallback for offline
+       display/Gazebo use where no live driver is publishing those frames. -->
   <xacro:sensor_d435
-    parent="camera_tilt_link"
+    parent="realsense_Link"
     name="camera"
     topics_ns="camera"
     use_nominal_extrinsics="$(arg use_nominal_extrinsics)"
     publish_pointcloud="$(arg publish_pointcloud)">
-    <origin xyz="0 0 0" rpy="0 ${camera_tilt_pitch} 0" />
+    <origin xyz="0 0 0" rpy="0 0 0" />
   </xacro:sensor_d435>
   <link

Commit message: reverted the realsense issue

File: ros_ws/src/nexzino/urdf/nexzino.urdf.xacro (robot description, xacro)
@@ -700,26 +700,44 @@
       xyz="0 0 0" />
   </joint>
-  <!-- Camera sensor frames attached directly at realsense_Link's own pose -
-       zero extra rotation, zero extra offset. realsense_Link's mesh (a
-       combined mount-arm + camera unit, confirmed visually against the
-       real robot) IS the ground truth for where/how the camera sits; no
-       hand-derived compensating rotation on top of it. (An earlier attempt
-       to derive that compensating rotation mathematically produced a
-       provably wrong result - the mesh mixes mount-arm and camera geometry,
-       so its own axes can't be read off computationally either. This is
-       the deliberate alternative: trust the CAD pose completely instead of
-       guessing a correction for it.)
-       Depth/color/optical frame orientations still come from the live
-       camera driver's own calibrated extrinsics (realsense_bringup.launch's
-       publish_tf:=true / use_nominal_extrinsics:=false), not static numbers
-       here - use_nominal_extrinsics is kept as a fallback for offline
-       display/Gazebo use where no live driver is publishing those frames. -->
+  <!-- camera_tilt_link re-establishes standard camera-body convention
+       (X=forward, Y=left, Z=up) on top of realsense_Link's own frame - this
+       exact rotation (1.5708, 3.1416, 3.1416) is the one already proven, by
+       explicit rotation-matrix calculation, to make a camera attached here
+       read out exactly forward-level. It is NOT a guess.
+       camera_tilt_pitch below is the one remaining unknown: the physical
+       camera is mounted tilted down by some angle, confirmed by loading the
+       real CAD mesh (nexa package) - a plain screenshot comparison isn't
+       precise enough to read off the exact angle, so this defaults to 0
+       (matches the old, forward-level behavior) rather than guessing a
+       number. To find the real value: watch nav_console's live camera feed
+       (or RViz's point cloud) while adjusting this, positive tilts the
+       camera further DOWN (confirmed: positive pitch about Y in this frame
+       rotates +X toward -Z). Try increments like 0.2-0.5 (≈11-29°) and
+       rebuild until the floor fills the frame the way it does on the real
+       robot.
+       (A direct identity attachment to realsense_Link - trusting its raw
+       CAD pose with no compensating rotation at all - was tried and
+       reported only partially correct, so reverted back to this tunable
+       form.) -->
+  <xacro:property name="camera_tilt_pitch" value="0" />
+  <link name="camera_tilt_link" />
+  <joint name="camera_tilt_joint" type="fixed">
+    <origin xyz="0 0 0" rpy="1.5708 3.1416 3.1416" />
+    <parent link="realsense_Link" />
+    <child link="camera_tilt_link" />
+  </joint>
+  <!-- Depth/color/optical frame orientations come from the live camera
+       driver's own calibrated extrinsics (see realsense_bringup.launch's
+       publish_tf:=true / use_nominal_extrinsics:=false), not from static
+       numbers here - use_nominal_extrinsics is kept as a fallback for
+       offline display/Gazebo use where no live driver is publishing those
+       frames. -->
   <xacro:sensor_d435
-    parent="realsense_Link"
+    parent="camera_tilt_link"
     name="camera"
     topics_ns="camera"
     use_nominal_extrinsics="$(arg use_nominal_extrinsics)"
     publish_pointcloud="$(arg publish_pointcloud)">
-    <origin xyz="0 0 0" rpy="0 0 0" />
+    <origin xyz="0 0 0" rpy="0 ${camera_tilt_pitch} 0" />
   </xacro:sensor_d435>
   <link

Commit message: working basic

File: ros_ws/src/nexzino/urdf/nexzino.urdf.xacro (robot description, xacro)
@@ -720,5 +720,5 @@
        reported only partially correct, so reverted back to this tunable
        form.) -->
-  <xacro:property name="camera_tilt_pitch" value="0" />
+  <xacro:property name="camera_tilt_pitch" value="0.959931" />
   <link name="camera_tilt_link" />
   <joint name="camera_tilt_joint" type="fixed">
